Commit message: Added a neck for crying out loud.\nChanged paths to make life easier on the URDF loader. Will probably undo that change at some point.

File: model.urdf (robot description, URDF)
Before this commit: robot huboplus, 57 links, 56 joints
Links:
- removed link Body_HNP
- added link Body_Head, mass 0.374251; collision mesh filename=./meshes/Body_Head_col.dae; visual mesh filename=./meshes/Body_Head_vis.dae
- added link Body_Head_Empty
- added link Body_Neck; collision mesh filename=./meshes/Body_Neck_col.dae
- link Body_Hip: geometry collision mesh filename=./meshes/Body_Hip_col.dae; visual mesh filename=./meshes/Body_Hip_vis.dae
- link Body_LAP: geometry collision mesh filename=./meshes/Body_LAP_col.dae; visual mesh filename=./meshes/Body_LAP_vis.dae
- link Body_LAR: geometry collision mesh filename=./meshes/Body_LAR_col.dae; visual mesh filename=./meshes/Body_LAR_vis.dae
- link Body_LEP: geometry collision mesh filename=./meshes/Body_LEP_col.dae; visual mesh filename=./meshes/Body_LEP_vis.dae
- link Body_LHP: geometry collision mesh filename=./meshes/Body_LHP_col.dae; visual mesh filename=./meshes/Body_LHP_vis.dae
- link Body_LHR: geometry collision mesh filename=./meshes/Body_LHR_col.dae; visual mesh filename=./meshes/Body_LHR_vis.dae
- link Body_LHY: geometry collision mesh filename=./meshes/Body_LHY_col.dae; visual mesh filename=./meshes/Body_LHY_vis.dae
- link Body_LKP: geometry collision mesh filename=./meshes/Body_LKP_col.dae; visual mesh filename=./meshes/Body_LKP_vis.dae
- link Body_LSP: geometry collision mesh filename=./meshes/Body_LSP_col.dae; visual mesh filename=./meshes/Body_LSP_vis.dae
- link Body_LSR: geometry collision mesh filename=./meshes/Body_LSR_col.dae; visual mesh filename=./meshes/Body_LSR_vis.dae
- link Body_LSY: geometry collision mesh filename=./meshes/Body_LSY_col.dae; visual mesh filename=./meshes/Body_LSY_vis.dae
- link Body_LWP: geometry collision mesh filename=./meshes/Body_LWP_col.dae; visual mesh filename=./meshes/Body_LWP_vis.dae
- link Body_LWY: geometry collision mesh filename=./meshes/Body_LWY_col.dae; visual mesh filename=./meshes/Body_LWY_vis.dae
- link Body_RAP: geometry collision mesh filename=./meshes/Body_RAP_col.dae; visual mesh filename=./meshes/Body_RAP_vis.dae
- link Body_RAR: geometry collision mesh filename=./meshes/Body_RAR_col.dae; visual mesh filename=./meshes/Body_RAR_vis.dae
- link Body_REP: geometry collision mesh filename=./meshes/Body_REP_col.dae; visual mesh filename=./meshes/Body_REP_vis.dae
- link Body_RHP: geometry collision mesh filename=./meshes/Body_RHP_col.dae; visual mesh filename=./meshes/Body_RHP_vis.dae
- link Body_RHR: geometry collision mesh filename=./meshes/Body_RHR_col.dae; visual mesh filename=./meshes/Body_RHR_vis.dae
- link Body_RHY: geometry collision mesh filename=./meshes/Body_RHY_col.dae; visual mesh filename=./meshes/Body_RHY_vis.dae
- link Body_RKP: geometry collision mesh filename=./meshes/Body_RKP_col.dae; visual mesh filename=./meshes/Body_RKP_vis.dae
- link Body_RSP: geometry collision mesh filename=./meshes/Body_RSP_col.dae; visual mesh filename=./meshes/Body_RSP_vis.dae
- link Body_RSR: geometry collision mesh filename=./meshes/Body_RSR_col.dae; visual mesh filename=./meshes/Body_RSR_vis.dae
- link Body_RSY: geometry collision mesh filename=./meshes/Body_RSY_col.dae; visual mesh filename=./meshes/Body_RSY_vis.dae
- link Body_RWP: geometry collision mesh filename=./meshes/Body_RWP_col.dae; visual mesh filename=./meshes/Body_RWP_vis.dae
- link Body_RWY: geometry collision mesh filename=./meshes/Body_RWY_col.dae; visual mesh filename=./meshes/Body_RWY_vis.dae
- link Body_Torso: geometry collision mesh filename=./meshes/Body_Torso_col.dae; visual mesh filename=./meshes/Body_Torso_vis.dae
- link leftIndexDistal: geometry collision mesh filename=./meshes/leftIndexDistal_vis.dae; visual mesh filename=./meshes/leftIndexDistal_vis.dae
- link leftIndexMedial: geometry collision mesh filename=./meshes/leftIndexMedial_vis.dae; visual mesh filename=./meshes/leftIndexMedial_vis.dae
- link leftIndexProximal: geometry collision mesh filename=./meshes/leftIndexProximal_vis.dae; visual mesh filename=./meshes/leftIndexProximal_vis.dae
- link leftMiddleDistal: geometry collision mesh filename=./meshes/leftMiddleDistal_vis.dae; visual mesh filename=./meshes/leftMiddleDistal_vis.dae
- link leftMiddleMedial: geometry collision mesh filename=./meshes/leftMiddleMedial_vis.dae; visual mesh filename=./meshes/leftMiddleMedial_vis.dae
- link leftMiddleProximal: geometry collision mesh filename=./meshes/leftMiddleProximal_vis.dae; visual mesh filename=./meshes/leftMiddleProximal_vis.dae
- link leftPinkyDistal: geometry collision mesh filename=./meshes/leftPinkyDistal_vis.dae; visual mesh filename=./meshes/leftPinkyDistal_vis.dae
- link leftPinkyMedial: geometry collision mesh filename=./meshes/leftPinkyMedial_vis.dae; visual mesh filename=./meshes/leftPinkyMedial_vis.dae
- link leftPinkyProximal: geometry collision mesh filename=./meshes/leftPinkyProximal_vis.dae; visual mesh filename=./meshes/leftPinkyProximal_vis.dae
- link leftRingDistal: geometry collision mesh filename=./meshes/leftRingDistal_vis.dae; visual mesh filename=./meshes/leftRingDistal_vis.dae
- link leftRingMedial: geometry collision mesh filename=./meshes/leftRingMedial_vis.dae; visual mesh filename=./meshes/leftRingMedial_vis.dae
- link leftRingProximal: geometry collision mesh filename=./meshes/leftRingProximal_vis.dae; visual mesh filename=./meshes/leftRingProximal_vis.dae
- link leftThumbDistal: geometry collision mesh filename=./meshes/leftThumbDistal_vis.dae; visual mesh filename=./meshes/leftThumbDistal_vis.dae
- link leftThumbMedial: geometry collision mesh filename=./meshes/leftThumbMedial_vis.dae; visual mesh filename=./meshes/leftThumbMedial_vis.dae
- link leftThumbProximal: geometry collision mesh filename=./meshes/leftThumbProximal_vis.dae; visual mesh filename=./meshes/leftThumbProximal_vis.dae
- link rightIndexDistal: geometry collision mesh filename=./meshes/rightIndexDistal_vis.dae; visual mesh filename=./meshes/rightIndexDistal_vis.dae
- link rightIndexMedial: geometry collision mesh filename=./meshes/rightIndexMedial_vis.dae; visual mesh filename=./meshes/rightIndexMedial_vis.dae
- link rightIndexProximal: geometry collision mesh filename=./meshes/rightIndexProximal_vis.dae; visual mesh filename=./meshes/rightIndexProximal_vis.dae
- link rightMiddleDistal: geometry collision mesh filename=./meshes/rightMiddleDistal_vis.dae; visual mesh filename=./meshes/rightMiddleDistal_vis.dae
- link rightMiddleMedial: geometry collision mesh filename=./meshes/rightMiddleMedial_vis.dae; visual mesh filename=./meshes/rightMiddleMedial_vis.dae
- link rightMiddleProximal: geometry collision mesh filename=./meshes/rightMiddleProximal_vis.dae; visual mesh filename=./meshes/rightMiddleProximal_vis.dae
- link rightPinkyDistal: geometry collision mesh filename=./meshes/rightPinkyDistal_vis.dae; visual mesh filename=./meshes/rightPinkyDistal_vis.dae
- link rightPinkyMedial: geometry collision mesh filename=./meshes/rightPinkyMedial_vis.dae; visual mesh filename=./meshes/rightPinkyMedial_vis.dae
- link rightPinkyProximal: geometry collision mesh filename=./meshes/rightPinkyProximal_vis.dae; visual mesh filename=./meshes/rightPinkyProximal_vis.dae
- link rightRingDistal: geometry collision mesh filename=./meshes/rightRingDistal_vis.dae; visual mesh filename=./meshes/rightRingDistal_vis.dae
- link rightRingMedial: geometry collision mesh filename=./meshes/rightRingMedial_vis.dae; visual mesh filename=./meshes/rightRingMedial_vis.dae
- link rightRingProximal: geometry collision mesh filename=./meshes/rightRingProximal_vis.dae; visual mesh filename=./meshes/rightRingProximal_vis.dae
- link rightThumbDistal: geometry collision mesh filename=./meshes/rightThumbDistal_vis.dae; visual mesh filename=./meshes/rightThumbDistal_vis.dae
- link rightThumbMedial: geometry collision mesh filename=./meshes/rightThumbMedial_vis.dae; visual mesh filename=./meshes/rightThumbMedial_vis.dae
- link rightThumbProximal: geometry collision mesh filename=./meshes/rightThumbProximal_vis.dae; visual mesh filename=./meshes/rightThumbProximal_vis.dae
Joints:
- removed joint HPY
- removed joint Knuckle2
- removed joint Knuckle212
- removed joint Knuckle215
- removed joint Knuckle218
- removed joint Knuckle221
- removed joint Knuckle230
- removed joint Knuckle233
- removed joint Knuckle236
- removed joint Knuckle239
- removed joint Knuckle29
- removed joint Knuckle3
- removed joint Knuckle310
- removed joint Knuckle313
- removed joint Knuckle316
- removed joint Knuckle319
- removed joint Knuckle322
- removed joint Knuckle331
- removed joint Knuckle334
- removed joint Knuckle337
- removed joint Knuckle340
- added joint HNR: type revolute, parent Body_Head_Empty, child Body_Head, origin xyz=0 0 0 rpy=0 -0 0, axis 1 0 0, limit lower=-0.523599 upper=0.523599 effort=10.0 velocity=1.0
- added joint NKY: type revolute, parent Body_Torso, child Body_Neck, origin xyz=0.0137246 0.0 0.1092625 rpy=0 -0 0, axis 0 0 1, limit lower=-1.5 upper=1.5 effort=10.0 velocity=1.0
- added joint WST: type revolute, parent Body_Torso, child Body_Hip, origin xyz=0.0122662 0.00245974 -0.15262 rpy=0 -0 0, axis 0 0 -1, limit lower=-3.14158 upper=3.14158 effort=10.0 velocity=1.0
- added joint leftIndexKnuckle2: type revolute, parent leftIndexProximal, child leftIndexMedial, origin xyz=0.032 0 0 rpy=0 -0 0, axis 0 0 -1, limit lower=-3.14 upper=3.14 effort=10.0 velocity=1.0
- added joint leftIndexKnuckle3: type revolute, parent leftIndexMedial, child leftIndexDistal, origin xyz=0.022 0 0 rpy=0 -0 0, axis 0 0 -1, limit lower=-3.14 upper=3.14 effort=10.0 velocity=1.0
- added joint leftMiddleKnuckle2: type revolute, parent leftMiddleProximal, child leftMiddleMedial, origin xyz=0.032 0 0 rpy=0 -0 0, axis 0 0 -1, limit lower=-3.14 upper=3.14 effort=10.0 velocity=1.0
- added joint leftMiddleKnuckle3: type revolute, parent leftMiddleMedial, child leftMiddleDistal, origin xyz=0.022 0 0 rpy=0 -0 0, axis 0 0 -1, limit lower=-3.14 upper=3.14 effort=10.0 velocity=1.0
- added joint leftPinkyKnuckle2: type revolute, parent leftPinkyProximal, child leftPinkyMedial, origin xyz=0.032 0 0 rpy=0 -0 0, axis 0 0 -1, limit lower=-3.14 upper=3.14 effort=10.0 velocity=1.0
- added joint leftPinkyKnuckle3: type revolute, parent leftPinkyMedial, child leftPinkyDistal, origin xyz=0.022 0 0 rpy=0 -0 0, axis 0 0 -1, limit lower=-3.14 upper=3.14 effort=10.0 velocity=1.0
- added joint leftRingKnuckle2: type revolute, parent leftRingProximal, child leftRingMedial, origin xyz=0.032 0 0 rpy=0 -0 0, axis 0 0 -1, limit lower=-3.14 upper=3.14 effort=10.0 velocity=1.0
- added joint leftRingKnuckle3: type revolute, parent leftRingMedial, child leftRingDistal, origin xyz=0.022 0 0 rpy=0 -0 0, axis 0 0 -1, limit lower=-3.14 upper=3.14 effort=10.0 velocity=1.0
- added joint leftThumbKnuckle2: type revolute, parent leftThumbProximal, child leftThumbMedial, origin xyz=0.032 0 0 rpy=0 -0 0, axis 0 0 -1, limit lower=-3.14 upper=3.14 effort=10.0 velocity=1.0
- added joint leftThumbKnuckle3: type revolute, parent leftThumbMedial, child leftThumbDistal, origin xyz=0.022 0 0 rpy=0 -0 0, axis 0 0 -1, limit lower=-3.14 upper=3.14 effort=10.0 velocity=1.0
- added joint rightIndexKnuckle2: type revolute, parent rightIndexProximal, child rightIndexMedial, origin xyz=0.032 0 0 rpy=0 -0 0, axis 0 0 -1, limit lower=0 upper=1.57 effort=10.0 velocity=1.0
- added joint rightIndexKnuckle3: type revolute, parent rightIndexMedial, child rightIndexDistal, origin xyz=0.022 0 0 rpy=0 -0 0, axis 0 0 -1, limit lower=0 upper=1.57 effort=10.0 velocity=1.0
- added joint rightMiddleKnuckle2: type revolute, parent rightMiddleProximal, child rightMiddleMedial, origin xyz=0.032 0 0 rpy=0 -0 0, axis 0 0 -1, limit lower=0 upper=1.57 effort=10.0 velocity=1.0
- added joint rightMiddleKnuckle3: type revolute, parent rightMiddleMedial, child rightMiddleDistal, origin xyz=0.022 0 0 rpy=0 -0 0, axis 0 0 -1, limit lower=0 upper=1.57 effort=10.0 velocity=1.0
- added joint rightPinkyKnuckle2: type revolute, parent rightPinkyProximal, child rightPinkyMedial, origin xyz=0.032 0 0 rpy=0 -0 0, axis 0 0 -1, limit lower=0 upper=1.57 effort=10.0 velocity=1.0
- added joint rightPinkyKnuckle3: type revolute, parent rightPinkyMedial, child rightPinkyDistal, origin xyz=0.022 0 0 rpy=0 -0 0, axis 0 0 -1, limit lower=0 upper=1.57 effort=10.0 velocity=1.0
- added joint rightRingKnuckle2: type revolute, parent rightRingProximal, child rightRingMedial, origin xyz=0.032 0 0 rpy=0 -0 0, axis 0 0 -1, limit lower=0 upper=1.57 effort=10.0 velocity=1.0
- added joint rightRingKnuckle3: type revolute, parent rightRingMedial, child rightRingDistal, origin xyz=0.022 0 0 rpy=0 -0 0, axis 0 0 -1, limit lower=0 upper=1.57 effort=10.0 velocity=1.0
- added joint rightThumbKnuckle2: type revolute, parent rightThumbProximal, child rightThumbMedial, origin xyz=0.032 0 0 rpy=0 -0 0, axis 0 0 -1, limit lower=0 upper=1.57 effort=10.0 velocity=1.0
- added joint rightThumbKnuckle3: type revolute, parent rightThumbMedial, child rightThumbDistal, origin xyz=0.022 0 0 rpy=0 -0 0, axis 0 0 -1, limit lower=0 upper=1.57 effort=10.0 velocity=1.0
- joint HNP: child Body_HNP -> Body_Head_Empty; origin xyz=0.0122581 0.0024526 0.196935 rpy=0 -0 0 -> xyz=-0.0014665 0.0024526 0.0876725 rpy=0 -0 0; parent Body_Torso -> Body_Neck
- joint LSR: limit lower=-1.5708 upper=1.5708 effort=10.0 velocity=1.0 -> lower=0 upper=3.14158 effort=10.0 velocity=1.0
- joint RSR: limit lower=-1.5708 upper=1.5708 effort=10.0 velocity=1.0 -> lower=-3.14158 upper=0 effort=10.0 velocity=1.0
- joint leftIndexKnuckle1: axis 0 0 1 -> 0 0 -1
- joint leftMiddleKnuckle1: axis 0 0 1 -> 0 0 -1
- joint leftPinkyKnuckle1: axis 0 0 1 -> 0 0 -1
- joint leftRingKnuckle1: axis 0 0 1 -> 0 0 -1
- joint leftThumbKnuckle1: axis 0 0 1 -> 0 0 -1
- joint rightIndexKnuckle1: axis 0 0 1 -> 0 0 -1; limit lower=-3.14 upper=3.14 effort=10.0 velocity=1.0 -> lower=0 upper=1.57 effort=10.0 velocity=1.0
- joint rightMiddleKnuckle1: axis 0 0 1 -> 0 0 -1; limit lower=-3.14 upper=3.14 effort=10.0 velocity=1.0 -> lower=0 upper=1.57 effort=10.0 velocity=1.0
- joint rightPinkyKnuckle1: axis 0 0 1 -> 0 0 -1; limit lower=-3.14 upper=3.14 effort=10.0 velocity=1.0 -> lower=0 upper=1.57 effort=10.0 velocity=1.0
- joint rightRingKnuckle1: axis 0 0 1 -> 0 0 -1; limit lower=-3.14 upper=3.14 effort=10.0 velocity=1.0 -> lower=0 upper=1.57 effort=10.0 velocity=1.0
- joint rightThumbKnuckle1: axis 0 0 1 -> 0 0 -1; limit lower=-3.14 upper=3.14 effort=10.0 velocity=1.0 -> lower=0 upper=1.57 effort=10.0 velocity=1.0

Commit message: Changed elbow and knee names to match hubo-ach.

File: model.urdf (robot description, URDF)
Before this commit: robot huboplus, 59 links, 58 joints
Links:
- removed link Body_LEP
- removed link Body_LKP
- removed link Body_REP
- removed link Body_RKP
- added link Body_LEB, mass 0.44094; collision mesh filename=./meshes/Body_LEB_col.dae; visual mesh filename=./meshes/Body_LEB_vis.dae
- added link Body_LKN, mass 1.80912; collision mesh filename=./meshes/Body_LKN_col.dae; visual mesh filename=./meshes/Body_LKN_vis.dae
- added link Body_REB, mass 0.44094; collision mesh filename=./meshes/Body_REB_col.dae; visual mesh filename=./meshes/Body_REB_vis.dae
- added link Body_RKN, mass 1.80912; collision mesh filename=./meshes/Body_RKN_col.dae; visual mesh filename=./meshes/Body_RKN_vis.dae
Joints:
- removed joint LEP
- removed joint LKP
- removed joint REP
- removed joint RKP
- added joint LEB: type revolute, parent Body_LSY, child Body_LEB, origin xyz=0.0219936 -0.018 -0.157505 rpy=0 -0 0, axis 0 1 0, limit lower=-2.49582 upper=0.0698132 effort=10.0 velocity=1.0
- added joint LKN: type revolute, parent Body_LHP, child Body_LKN, origin xyz=0.000766364 -0.0445011 -0.280007 rpy=0 -0 0, axis 0 1 0, limit lower=-0.0698132 upper=2.60054 effort=10.0 velocity=1.0
- added joint REB: type revolute, parent Body_RSY, child Body_REB, origin xyz=0.0219936 0.018 -0.157505 rpy=0 -0 0, axis 0 1 0, limit lower=-2.49582 upper=0.0698132 effort=10.0 velocity=1.0
- added joint RKN: type revolute, parent Body_RHP, child Body_RKN, origin xyz=0.000766364 0.0445011 -0.280007 rpy=0 -0 0, axis 0 1 0, limit lower=-0.0698132 upper=2.60054 effort=10.0 velocity=1.0
- joint LAP: parent Body_LKP -> Body_LKN
- joint LWY: parent Body_LEP -> Body_LEB
- joint RAP: parent Body_RKP -> Body_RKN
- joint RWY: parent Body_REP -> Body_REB

Commit message: New head model.

File: model.urdf (robot description, URDF)
Before this commit: robot huboplus, 59 links, 58 joints
Links:
- link Body_Head: geometry collision mesh filename=./meshes/Body_Head.stl; visual mesh filename=./meshes/Body_Head.stl

Commit message: Removed redundant finger Collada models

File: model.urdf (robot description, URDF)
Before this commit: robot huboplus, 59 links, 58 joints
Links:
- link leftIndexDistal: geometry collision mesh filename=./meshes/medial_distal.dae; visual mesh filename=./meshes/medial_distal.dae
- link leftIndexMedial: geometry collision mesh filename=./meshes/medial_distal.dae; visual mesh filename=./meshes/medial_distal.dae
- link leftIndexProximal: geometry collision mesh filename=./meshes/proximal.dae; visual mesh filename=./meshes/proximal.dae
- link leftMiddleDistal: geometry collision mesh filename=./meshes/medial_distal.dae; visual mesh filename=./meshes/medial_distal.dae
- link leftMiddleMedial: geometry collision mesh filename=./meshes/medial_distal.dae; visual mesh filename=./meshes/medial_distal.dae
- link leftMiddleProximal: geometry collision mesh filename=./meshes/proximal.dae; visual mesh filename=./meshes/proximal.dae
- link leftPinkyDistal: geometry collision mesh filename=./meshes/medial_distal.dae; visual mesh filename=./meshes/medial_distal.dae
- link leftPinkyMedial: geometry collision mesh filename=./meshes/medial_distal.dae; visual mesh filename=./meshes/medial_distal.dae
- link leftPinkyProximal: geometry collision mesh filename=./meshes/proximal.dae; visual mesh filename=./meshes/proximal.dae
- link leftRingDistal: geometry collision mesh filename=./meshes/medial_distal.dae; visual mesh filename=./meshes/medial_distal.dae
- link leftRingMedial: geometry collision mesh filename=./meshes/medial_distal.dae; visual mesh filename=./meshes/medial_distal.dae
- link leftRingProximal: geometry collision mesh filename=./meshes/proximal.dae; visual mesh filename=./meshes/proximal.dae
- link leftThumbDistal: geometry collision mesh filename=./meshes/medial_distal.dae; visual mesh filename=./meshes/medial_distal.dae
- link leftThumbMedial: geometry collision mesh filename=./meshes/medial_distal.dae; visual mesh filename=./meshes/medial_distal.dae
- link leftThumbProximal: geometry collision mesh filename=./meshes/proximal.dae; visual mesh filename=./meshes/proximal.dae
- link rightIndexDistal: geometry collision mesh filename=./meshes/medial_distal.dae; visual mesh filename=./meshes/medial_distal.dae
- link rightIndexMedial: geometry collision mesh filename=./meshes/medial_distal.dae; visual mesh filename=./meshes/medial_distal.dae
- link rightIndexProximal: geometry collision mesh filename=./meshes/proximal.dae; visual mesh filename=./meshes/proximal.dae
- link rightMiddleDistal: geometry collision mesh filename=./meshes/medial_distal.dae; visual mesh filename=./meshes/medial_distal.dae
- link rightMiddleMedial: geometry collision mesh filename=./meshes/medial_distal.dae; visual mesh filename=./meshes/medial_distal.dae
- link rightMiddleProximal: geometry collision mesh filename=./meshes/proximal.dae; visual mesh filename=./meshes/proximal.dae
- link rightPinkyDistal: geometry collision mesh filename=./meshes/medial_distal.dae; visual mesh filename=./meshes/medial_distal.dae
- link rightPinkyMedial: geometry collision mesh filename=./meshes/medial_distal.dae; visual mesh filename=./meshes/medial_distal.dae
- link rightPinkyProximal: geometry collision mesh filename=./meshes/proximal.dae; visual mesh filename=./meshes/proximal.dae
- link rightRingDistal: geometry collision mesh filename=./meshes/medial_distal.dae; visual mesh filename=./meshes/medial_distal.dae
- link rightRingMedial: geometry collision mesh filename=./meshes/medial_distal.dae; visual mesh filename=./meshes/medial_distal.dae
- link rightRingProximal: geometry collision mesh filename=./meshes/proximal.dae; visual mesh filename=./meshes/proximal.dae
- link rightThumbDistal: geometry collision mesh filename=./meshes/medial_distal.dae; visual mesh filename=./meshes/medial_distal.dae
- link rightThumbMedial: geometry collision mesh filename=./meshes/medial_distal.dae; visual mesh filename=./meshes/medial_distal.dae
- link rightThumbProximal: geometry collision mesh filename=./meshes/proximal.dae; visual mesh filename=./meshes/proximal.dae
